Commit message: gazeboに入れる直前(rviz表示可能)

File: awagv_description/urdf/awagv.xacro (robot description, xacro)
@@ -13,23 +13,23 @@
   <xacro:property name="RIGHT_ANGLE" value="1.570796327"/>
   <!-- Used for fixing robot to Gazebo 'base_link' -->
-  <link name="base_link"/>
+  <link name="base_footprint"/>
   <joint name="fixed" type="fixed">
-    <parent link="base_link"/>
-    <child link="body_link"/>
+    <parent link="base_footprint"/>
+    <child link="base_link"/>
   </joint>
-<!-- ==================================================================body_link -->
-  <link name="body_link">
+  <!-- ==================================================================body_link -->
+  <link name="base_link">
     <visual>
-        <origin xyz="0 0 0" rpy="0 0 0"/>
-        <axis xyz="0 0 0"/>
-        <geometry>
-          <mesh filename="package://awagv_description/meshes/awagv.stl" scale="1 1 1"/>
-        </geometry>
-        <material name="grey"/>
+      <origin xyz="0 0 0" rpy="0 0 0"/>
+      <axis xyz="0 0 0"/>
+      <geometry>
+        <mesh filename="package://awagv_description/meshes/awagv.stl" scale="1 1 1"/>
+      </geometry>
+      <material name="grey"/>
     </visual>
   </link>
 <!-- +++++++++++++++++++++++++++++++++++++++++++++++++++++++++++++++++joint_wheel_r -->
     <joint name="wheel_r_joint" type="continuous">
-      <parent link="body_link"/>
+      <parent link="base_link"/>
       <child link="wheel_link_r"/>
       <origin xyz="0.28 0 0.055" rpy="0 0 ${-RIGHT_ANGLE}"/>
@@ -39,5 +39,5 @@
 <!-- +++++++++++++++++++++++++++++++++++++++++++++++++++++++++++++++++joint_wheel_l -->
     <joint name="wheel_l_joint" type="continuous">
-      <parent link="body_link"/>
+      <parent link="base_link"/>
       <child link="wheel_link_l"/>
       <origin xyz="-0.28 0 0.055" rpy="0 0 ${RIGHT_ANGLE}"/>
@@ -65,18 +65,3 @@
         </visual>
     </link>
-  <!-- ************ Gazebo Transmission ********************* -->
-  <xacro:wheel_trans_v0 prefix="right" />
-  <xacro:wheel_trans_v0 prefix="left" />
-  <gazebo>
-    <plugin name="gazebo_ros_control" filename="libgazebo_ros_control.so">
-    </plugin>
-  </gazebo>
-  <!-- ********* Gazebo Base ******* -->
-  <xacro:base_gazebo_v0/>
-  <xacro:wheel_gazebo_v0 prefix="right"/>
-  <xacro:wheel_gazebo_v0 prefix="left"/>
-  <xacro:wheel_gazebo_control_v0 rate="25"/>
-  <xacro:lrf_gazebo_v0 prefix="front"
-    min_rad="-1.65806278939" max_rad="1.65806278939"
-    min_range="0.10" max_range="5.0"/>
 </robot>

Commit message: gazebo用launch作成直前。rviz起動確認

File: awagv_description/urdf/awagv.xacro (robot description, xacro)
@@ -13,5 +13,10 @@
   <xacro:property name="RIGHT_ANGLE" value="1.570796327"/>
   <!-- Used for fixing robot to Gazebo 'base_link' -->
-  <link name="base_footprint"/>
+  <link name="base_footprint">
+    <origin xyz="0 0 0"/>
+  </link>
+  <gazebo reference="base_footprint">
+    <turnGravityOff>false</turnGravityOff>
+  </gazebo>
   <joint name="fixed" type="fixed">
     <parent link="base_footprint"/>
@@ -26,4 +31,8 @@
         <mesh filename="package://awagv_description/meshes/awagv.stl" scale="1 1 1"/>
       </geometry>
+      <inertial>
+        <mass value="18.85" />
+        <inertia ixx="1.009" ixy="0.064" ixz="0.095" iyy="0.818" iyz="-0.344" izz="0.867"/>
+      </inertial>
       <material name="grey"/>
     </visual>
@@ -37,4 +46,15 @@
       <dynamics damping="0.7"/>
     </joint>
+<!-- ****************************************************************Transmission wheel_r -->
+  <transmission name="right_wheel_trans">
+    <type>transmission_interface/SimpleTransmission</type>
+    <joint name="wheel_r_joint">
+      <hardwareInterface>VelocityJointInterface</hardwareInterface>
+    </joint>
+    <actuator name="left_wheel_motor">
+      <hardwareInterface>VelocityJointInterface</hardwareInterface>
+      <mechanicalReduction>30</mechanicalReduction>
+    </actuator>
+  </transmission>
 <!-- +++++++++++++++++++++++++++++++++++++++++++++++++++++++++++++++++joint_wheel_l -->
     <joint name="wheel_l_joint" type="continuous">
@@ -45,4 +65,35 @@
       <dynamics damping="0.7"/>
     </joint>
+<!-- ****************************************************************Transmission wheel_r -->
+  <transmission name="left_wheel_trans">
+    <type>transmission_interface/SimpleTransmission</type>
+    <joint name="wheel_l_joint">
+      <hardwareInterface>VelocityJointInterface</hardwareInterface>
+    </joint>
+    <actuator name="left_wheel_motor">
+      <hardwareInterface>VelocityJointInterface</hardwareInterface>
+      <mechanicalReduction>30</mechanicalReduction>
+    </actuator>
+  </transmission>
+  <gazebo>
+    <plugin name="gazebo_ros_control" filename="libgazebo_ros_control.so">
+      <robotNamespace>awagv</robotNamespace>
+    </plugin>
+  </gazebo>
+  <gazebo reference="base_link">
+    <selfCollide>true</selfCollide>
+    <mu1 value="0.05"/>
+    <mu2 value="0.05"/>
+  </gazebo>
+  <gazebo reference="wheel_link_l">
+    <selfCollide>true</selfCollide>
+    <mu1 value="0.8"/>
+    <mu2 value="0.8"/>
+  </gazebo>
+  <gazebo reference="wheel_link_r">
+    <selfCollide>true</selfCollide>
+    <mu1 value="0.8"/>
+    <mu2 value="0.8"/>
+  </gazebo>
 <!-- ==================================================================link_wheel -->
     <link name="wheel_link_r">

Commit message: Gazebo + rviz + awagv 起動確認

File: awagv_description/urdf/awagv.xacro (robot description, xacro)
@@ -2,78 +2,127 @@
 <!-- Revolute-Revolute Manipulator -->
 <robot name="awagv" xmlns:xacro="http://www.ros.org/wiki/xacro">
-<!-- Rviz colors -->
-  <material name="grey">
-    <color rgba="0.2 0.2 0.2 1.0"/>
-  </material>
-  <material name="orange">
-    <color rgba="${255/255} ${108/255} ${10/255} 1.0"/>
-  </material>
-  <!-- Constants for robot dimensions -->
   <xacro:property name="PI" value="3.1415926535897931"/>
   <xacro:property name="RIGHT_ANGLE" value="1.570796327"/>
-  <!-- Used for fixing robot to Gazebo 'base_link' -->
-  <link name="base_footprint">
-    <origin xyz="0 0 0"/>
-  </link>
-  <gazebo reference="base_footprint">
-    <turnGravityOff>false</turnGravityOff>
-  </gazebo>
-  <joint name="fixed" type="fixed">
-    <parent link="base_footprint"/>
-    <child link="base_link"/>
-  </joint>
-  <!-- ==================================================================body_link -->
   <link name="base_link">
     <visual>
-      <origin xyz="0 0 0" rpy="0 0 0"/>
-      <axis xyz="0 0 0"/>
+      <geometry>
+        <mesh filename="package://awagv_description/meshes/awagv.stl" scale="1 1 1" />
+      </geometry>
+    </visual>
+    <collision>
       <geometry>
         <mesh filename="package://awagv_description/meshes/awagv.stl" scale="1 1 1"/>
       </geometry>
-      <inertial>
-        <mass value="18.85" />
-        <inertia ixx="1.009" ixy="0.064" ixz="0.095" iyy="0.818" iyz="-0.344" izz="0.867"/>
-      </inertial>
-      <material name="grey"/>
+    </collision>
+   <inertial>
+    <origin xyz="0 0 0"/>
+    <mass value="15.0"/>
+    <inertia ixx="0.1" ixy="0" ixz="0" iyy="0.1" iyz="0" izz="0.1"/>
+   </inertial>
+  </link>
+  <link name="left_wheel_link">
+    <visual>
+      <geometry>
+        <mesh filename="package://awagv_description/meshes/agvwheel.stl" scale="1 1 1"/>
+      </geometry>
+      <origin xyz="0 0 0" rpy="0 0 0"/>
+      <material name="black"/>
     </visual>
+    <collision>
+      <geometry>
+        <mesh filename="package://awagv_description/meshes/agvwheel.stl" scale="1 1 1"/>
+      </geometry>
+    </collision>
+   <inertial>
+    <origin xyz="0 0 0"/>
+    <mass value="1"/>
+    <inertia ixx="0.1" ixy="0" ixz="0" iyy="0.1" iyz="0" izz="0.1"/>
+   </inertial>
   </link>
-<!-- +++++++++++++++++++++++++++++++++++++++++++++++++++++++++++++++++joint_wheel_r -->
-    <joint name="wheel_r_joint" type="continuous">
-      <parent link="base_link"/>
-      <child link="wheel_link_r"/>
-      <origin xyz="0.28 0 0.055" rpy="0 0 ${-RIGHT_ANGLE}"/>
-      <axis xyz="0 1 0"/>
-      <dynamics damping="0.7"/>
-    </joint>
-<!-- ****************************************************************Transmission wheel_r -->
-  <transmission name="right_wheel_trans">
-    <type>transmission_interface/SimpleTransmission</type>
-    <joint name="wheel_r_joint">
-      <hardwareInterface>VelocityJointInterface</hardwareInterface>
-    </joint>
-    <actuator name="left_wheel_motor">
-      <hardwareInterface>VelocityJointInterface</hardwareInterface>
-      <mechanicalReduction>30</mechanicalReduction>
-    </actuator>
-  </transmission>
-<!-- +++++++++++++++++++++++++++++++++++++++++++++++++++++++++++++++++joint_wheel_l -->
-    <joint name="wheel_l_joint" type="continuous">
-      <parent link="base_link"/>
-      <child link="wheel_link_l"/>
-      <origin xyz="-0.28 0 0.055" rpy="0 0 ${RIGHT_ANGLE}"/>
-      <axis xyz="0 1 0"/>
-      <dynamics damping="0.7"/>
-    </joint>
-<!-- ****************************************************************Transmission wheel_r -->
-  <transmission name="left_wheel_trans">
-    <type>transmission_interface/SimpleTransmission</type>
-    <joint name="wheel_l_joint">
-      <hardwareInterface>VelocityJointInterface</hardwareInterface>
-    </joint>
-    <actuator name="left_wheel_motor">
-      <hardwareInterface>VelocityJointInterface</hardwareInterface>
-      <mechanicalReduction>30</mechanicalReduction>
-    </actuator>
-  </transmission>
+  <joint name="left_wheel_joint" type="continuous">
+    <parent link="base_link"/>
+    <child link="left_wheel_link"/>
+    <origin xyz="-0.28 0 0.055" rpy="0 0 ${RIGHT_ANGLE}"/>
+    <axis xyz="0 1 0"/>
+  </joint>
+  <link name="right_wheel_link">
+    <visual>
+      <geometry>
+        <mesh filename="package://awagv_description/meshes/agvwheel.stl" scale="1 1 1"/>
+      </geometry>
+      <origin xyz="0 0 0" rpy="0 0 ${-RIGHT_ANGLE*2}"/>
+      <axis xyz="0 0 0"/>
+      <material name="black"/>
+    </visual>
+    <collision>
+      <geometry>
+        <mesh filename="package://awagv_description/meshes/agvwheel.stl" scale="1 1 1"/>
+      </geometry>
+    </collision>
+   <inertial>
+      <origin xyz="0 0 0"/>
+      <mass value="1"/>
+      <inertia ixx="0.1" ixy="0" ixz="0" iyy="0.1" iyz="0" izz="0.1"/>
+   </inertial>
+  </link>
+  <joint name="right_wheel_joint" type="continuous">
+    <parent link="base_link"/>
+    <child link="right_wheel_link"/>
+    <origin xyz="0.28 0 0.055" rpy="0 0 ${RIGHT_ANGLE}"/>
+    <axis xyz="0 1 0"/>
+  </joint>
+  <link name="caster_link">
+    <visual>
+      <geometry>
+        <sphere radius="0.055"/>
+      </geometry>
+      <material name="green">
+        <color rgba="0 1 0 1"/>
+      </material>
+    </visual>
+    <collision>
+      <geometry>
+        <sphere radius="0.055"/>
+      </geometry>
+    </collision>
+   <inertial>
+    <origin xyz="0 0 0"/>
+    <mass value="0.500"/>
+    <inertia ixx="0.0001" ixy="0" ixz="0" iyy="0.0001"  iyz="0" izz="0.0001"/>
+   </inertial>
+  </link>
+  <joint name="caster_joint" type="fixed">
+   <parent link="base_link"/>
+   <child link="caster_link"/>
+   <origin xyz="0 0.2 0.055"/>
+ </joint>
+ <link name="base_footprint"/>
+  <joint name="base_link_joint" type="fixed">
+   <parent link="base_footprint"/>
+   <child link="base_link"/>
+   <origin xyz="0 0 0" rpy="0 0 ${-RIGHT_ANGLE}"/>
+ </joint>
+  <!-- ===============  Transmission =============== -->
+<transmission name="left_wheel_trans">
+  <type>transmission_interface/SimpleTransmission</type>
+  <joint name="left_wheel_joint">
+    <hardwareInterface>VelocityJointInterface</hardwareInterface>
+  </joint>
+  <actuator name="left_wheel_motor">
+    <hardwareInterface>VelocityJointInterface</hardwareInterface>
+    <mechanicalReduction>30</mechanicalReduction>
+  </actuator>
+</transmission>
+<transmission name="right_wheel_trans">
+  <type>transmission_interface/SimpleTransmission</type>
+  <joint name="right_wheel_joint">
+    <hardwareInterface>VelocityJointInterface</hardwareInterface>
+  </joint>
+  <actuator name="right_wheel_motor">
+    <hardwareInterface>VelocityJointInterface</hardwareInterface>
+    <mechanicalReduction>30</mechanicalReduction>
+  </actuator>
+</transmission>
+  <!-- =============== Gazebo =============== -->
   <gazebo>
     <plugin name="gazebo_ros_control" filename="libgazebo_ros_control.so">
@@ -81,38 +130,24 @@
     </plugin>
   </gazebo>
-  <gazebo reference="base_link">
-    <selfCollide>true</selfCollide>
-    <mu1 value="0.05"/>
-    <mu2 value="0.05"/>
+ <gazebo reference="base_link">
+   <selfCollide>true</selfCollide>
+    <mu1 value="0.05" />
+    <mu2 value="0.05" />
   </gazebo>
-  <gazebo reference="wheel_link_l">
-    <selfCollide>true</selfCollide>
-    <mu1 value="0.8"/>
-    <mu2 value="0.8"/>
+ <gazebo reference="left_wheel_link">
+   <selfCollide>true</selfCollide>
+    <mu1 value="1.0" />
+    <mu2 value="1.0" />
   </gazebo>
-  <gazebo reference="wheel_link_r">
-    <selfCollide>true</selfCollide>
-    <mu1 value="0.8"/>
-    <mu2 value="0.8"/>
+ <gazebo reference="right_wheel_link">
+   <selfCollide>true</selfCollide>
+    <mu1 value="1.0" />
+    <mu2 value="1.0" />
   </gazebo>
-<!-- ==================================================================link_wheel -->
-    <link name="wheel_link_r">
-        <visual>
-          <origin xyz="0 0 0" rpy="0 0 0"/>
-          <geometry>
-            <mesh filename="package://awagv_description/meshes/agvwheel.stl" scale="1 1 1"/>
-          </geometry>
-          <material name="orange"/>
-        </visual>
-    </link>
-<!-- ==================================================================link_wheel -->
-    <link name="wheel_link_l">
-        <visual>
-          <origin xyz="0 0 0" rpy="0 0 0"/>
-          <geometry>
-            <mesh filename="package://awagv_description/meshes/agvwheel.stl" scale="1 1 1"/>
-          </geometry>
-          <material name="orange"/>
-        </visual>
-    </link>
+ <gazebo reference="caster_link">
+   <selfCollide>true</selfCollide>
+     <!-- This caster is no frictional resistance. -->
+    <mu1 value="0.0" />
+    <mu2 value="0.0" />
+  </gazebo>
 </robot>

Commit message: Gazebo + rviz + PS3Joy

File: awagv_description/urdf/awagv.xacro (robot description, xacro)
@@ -16,7 +16,7 @@
     </collision>
    <inertial>
-    <origin xyz="0 0 0"/>
-    <mass value="15.0"/>
-    <inertia ixx="0.1" ixy="0" ixz="0" iyy="0.1" iyz="0" izz="0.1"/>
+    <origin xyz="0.0 0.0 0.1675218"/>
+    <mass value="14.84863433"/>
+    <inertia ixx="0.000000388" ixy="-0.000000015" ixz="-0.000000071" iyy="0.000000414" iyz="-0.00000002" izz="0.000000675"/>
    </inertial>
   </link>
@@ -72,9 +72,10 @@
     <axis xyz="0 1 0"/>
   </joint>
-  <link name="caster_link">
+  <link name="caster_link_fl">
     <visual>
       <geometry>
-        <sphere radius="0.055"/>
+        <sphere radius="0.035" />
       </geometry>
+      <origin xyz="0 0 0" rpy="0 ${RIGHT_ANGLE} 0"/>
       <material name="green">
         <color rgba="0 1 0 1"/>
@@ -83,18 +84,46 @@
     <collision>
       <geometry>
-        <sphere radius="0.055"/>
+        <sphere radius="0.035" />
       </geometry>
+      <origin xyz="0 0 0" rpy="0 ${RIGHT_ANGLE} 0"/>
     </collision>
-   <inertial>
-    <origin xyz="0 0 0"/>
-    <mass value="0.500"/>
-    <inertia ixx="0.0001" ixy="0" ixz="0" iyy="0.0001"  iyz="0" izz="0.0001"/>
-   </inertial>
+    <inertial>
+      <origin xyz="0 0 0"/>
+      <mass value="0.500"/>
+      <inertia ixx="0.0001" ixy="0" ixz="0" iyy="0.0001"  iyz="0" izz="0.0001"/>
+    </inertial>
   </link>
-  <joint name="caster_joint" type="fixed">
-   <parent link="base_link"/>
-   <child link="caster_link"/>
-   <origin xyz="0 0.2 0.055"/>
- </joint>
+  <link name="caster_link_rr">
+    <visual>
+      <geometry>
+        <sphere radius="0.035" />
+      </geometry>
+      <origin xyz="0 0 0" rpy="0 ${RIGHT_ANGLE} 0"/>
+      <material name="green">
+        <color rgba="0 1 0 1"/>
+      </material>
+    </visual>
+    <collision>
+      <geometry>
+        <sphere radius="0.035" />
+      </geometry>
+      <origin xyz="0 0 0" rpy="0 ${RIGHT_ANGLE} 0"/>
+    </collision>
+    <inertial>
+      <origin xyz="0 0 0"/>
+      <mass value="0.500"/>
+      <inertia ixx="0.0001" ixy="0" ixz="0" iyy="0.0001"  iyz="0" izz="0.0001"/>
+    </inertial>
+  </link>
+  <joint name="caster_joint_fl" type="fixed">
+    <parent link="base_link"/>
+    <child link="caster_link_fl"/>
+    <origin xyz="0 0.25 0.035"/>
+  </joint>
+  <joint name="caster_joint_rr" type="fixed">
+    <parent link="base_link"/>
+    <child link="caster_link_rr"/>
+    <origin xyz="0 -0.25 0.035"/>
+  </joint>
  <link name="base_footprint"/>
   <joint name="base_link_joint" type="fixed">
@@ -137,17 +166,23 @@
  <gazebo reference="left_wheel_link">
    <selfCollide>true</selfCollide>
-    <mu1 value="1.0" />
-    <mu2 value="1.0" />
+    <mu1 value="0.9" />
+    <mu2 value="0.9" />
   </gazebo>
  <gazebo reference="right_wheel_link">
    <selfCollide>true</selfCollide>
-    <mu1 value="1.0" />
-    <mu2 value="1.0" />
+    <mu1 value="0.9" />
+    <mu2 value="0.9" />
   </gazebo>
- <gazebo reference="caster_link">
-   <selfCollide>true</selfCollide>
-     <!-- This caster is no frictional resistance. -->
-    <mu1 value="0.0" />
-    <mu2 value="0.0" />
+  <gazebo reference="caster_link_fl">
+    <selfCollide>true</selfCollide>
+    <!-- This caster is no frictional resistance. -->
+    <mu1 value="0.05" />
+    <mu2 value="0.05" />
+  </gazebo>
+  <gazebo reference="caster_link_rr">
+    <selfCollide>true</selfCollide>
+    <!-- This caster is no frictional resistance. -->
+    <mu1 value="0.05" />
+    <mu2 value="0.05" />
   </gazebo>
 </robot>
